File: PCB/bare_mouse/bloo.kicad_pcb (KiCad board)
At the start: 2 copper layers, 0 parts

Commit message: Reviewed and updated schematics accordingly, updated BOM, created PCB Design Notes
Parts:
- added BT1: Battery_Cell, Connector_PinSocket_2.54mm:PinSocket_1x02_P2.54mm_Vertical, F.Cu at (98.0, 65.5)
- added BT_MH1: M2, MountingHole:MountingHole_2.2mm_M2, F.Cu at (18.2, 77.9)
- added BT_MH2: M2, MountingHole:MountingHole_2.2mm_M2, F.Cu at (18.2, 83.8)
- added BT_MH3: M2, MountingHole:MountingHole_2.2mm_M2, F.Cu at (24.1, 77.9)
- added BT_MH4: M2, MountingHole:MountingHole_2.2mm_M2, F.Cu at (24.1, 83.8)
- added BZ1: Buzzer, Buzzer_Beeper:MagneticBuzzer_PUI_AT-0927-TT-6-R, F.Cu at (54.1, 102.2)
- added C1: 0.1uF, Capacitor_SMD:C_1206_3216Metric_Pad1.33x1.80mm_HandSolder, F.Cu at (18.2, 88.5)
- added C10: 10uF(Tantalum), Capacitor_SMD:C_1206_3216Metric_Pad1.33x1.80mm_HandSolder, F.Cu at (18.2, 108.6)
- added C11: 10uF, Capacitor_SMD:C_1206_3216Metric_Pad1.33x1.80mm_HandSolder, F.Cu at (24.2, 88.5)
- added C12: 0.1uF, Capacitor_SMD:C_1206_3216Metric_Pad1.33x1.80mm_HandSolder, F.Cu at (24.2, 91.8)
- added C13: 0.1uF, Capacitor_SMD:C_1206_3216Metric_Pad1.33x1.80mm_HandSolder, F.Cu at (24.2, 95.2)
- added C14: 1uF, Capacitor_SMD:C_1206_3216Metric_Pad1.33x1.80mm_HandSolder, F.Cu at (24.2, 98.5)
- added C15: 1uF, Capacitor_SMD:C_1206_3216Metric_Pad1.33x1.80mm_HandSolder, F.Cu at (24.2, 101.9)
- added C16: 100uF, Capacitor_THT:CP_Radial_D6.3mm_P2.50mm, F.Cu at (98.5, 43.4)
- added C17: 1uF, Capacitor_SMD:C_1206_3216Metric_Pad1.33x1.80mm_HandSolder, F.Cu at (24.2, 105.2)
- added C18: 1uF, Capacitor_SMD:C_1206_3216Metric_Pad1.33x1.80mm_HandSolder, F.Cu at (24.2, 108.6)
- added C19: 0.1uF, Capacitor_SMD:C_1206_3216Metric_Pad1.33x1.80mm_HandSolder, F.Cu at (30.2, 88.5)
- added C2: 100uF, Capacitor_THT:CP_Radial_D6.3mm_P2.50mm, F.Cu at (98.5, 35.5)
- added C20: 1uF, Capacitor_SMD:C_1206_3216Metric_Pad1.33x1.80mm_HandSolder, F.Cu at (30.2, 91.8)
- added C21: 1uF, Capacitor_SMD:C_1206_3216Metric_Pad1.33x1.80mm_HandSolder, F.Cu at (30.2, 95.2)
- added C25: 10nF, Capacitor_SMD:C_1206_3216Metric_Pad1.33x1.80mm_HandSolder, F.Cu at (30.2, 98.5)
- added C3: 10uF, Capacitor_SMD:C_1206_3216Metric_Pad1.33x1.80mm_HandSolder, F.Cu at (18.2, 91.8)
- added C4: 0.1uF, Capacitor_SMD:C_1206_3216Metric_Pad1.33x1.80mm_HandSolder, F.Cu at (18.2, 95.2)
- added C5: 0.1uF, Capacitor_SMD:C_1206_3216Metric_Pad1.33x1.80mm_HandSolder, F.Cu at (18.2, 98.5)
- added C6: 22pF, Capacitor_SMD:C_0603_1608Metric_Pad1.08x0.95mm_HandSolder, F.Cu at (55.5, 76.2)
- added C7: 10uF, Capacitor_SMD:C_1206_3216Metric_Pad1.33x1.80mm_HandSolder, F.Cu at (18.2, 101.9)
- added C8: 22pF, Capacitor_SMD:C_0603_1608Metric_Pad1.08x0.95mm_HandSolder, F.Cu at (55.5, 78.7)
- added C9: 10uF, Capacitor_SMD:C_1206_3216Metric_Pad1.33x1.80mm_HandSolder, F.Cu at (18.2, 105.2)
- added D0: SFH4545, MM_Library:Emitter, F.Cu at (64.1, 72.4)
- added D1: SFH4545, MM_Library:Emitter, F.Cu at (69.7, 72.4)
- added D2: SFH4545, MM_Library:Emitter, F.Cu at (75.2, 72.4)
- added D3: SFH4545, MM_Library:Emitter, F.Cu at (80.8, 72.4)
- added D4: LED, LED_SMD:LED_0805_2012Metric_Pad1.15x1.40mm_HandSolder, F.Cu at (60.1, 76.4)
- added D5: LED, LED_SMD:LED_0805_2012Metric_Pad1.15x1.40mm_HandSolder, F.Cu at (60.1, 79.5)
- added D6: LED, LED_SMD:LED_0805_2012Metric_Pad1.15x1.40mm_HandSolder, F.Cu at (60.1, 82.5)
- added FB3: HZ0603C601R-10, Resistor_SMD:R_0603_1608Metric_Pad0.98x0.95mm_HandSolder, F.Cu at (55.5, 81.2)
- added FB4: HZ0603C601R-10, Resistor_SMD:R_0603_1608Metric_Pad0.98x0.95mm_HandSolder, F.Cu at (55.5, 83.7)
- added J1: Serial Debug Header, Connector_PinHeader_2.54mm:PinHeader_1x06_P2.54mm_Vertical, F.Cu at (88.7, 33.9)
- added J10: Conn_01x06_Female, Connector_PinSocket_2.54mm:PinSocket_1x06_P2.54mm_Vertical, F.Cu at (93.4, 33.9)
- added J2: SWD Header, Connector_PinHeader_2.54mm:PinHeader_1x05_P2.54mm_Vertical, F.Cu at (88.7, 51.2)
- added J4: Conn_ARM_JTAG_SWD_10, Connector_PinHeader_1.27mm:PinHeader_2x05_P1.27mm_Vertical, F.Cu at (96.0, 103.6)
- added J5: SWD Header, Connector_PinHeader_2.54mm:PinHeader_1x05_P2.54mm_Vertical, F.Cu at (93.4, 51.2)
- added JP1: JP_SWO, Jumper:SolderJumper-2_P1.3mm_Open_Pad1.0x1.5mm, F.Cu at (97.9, 50.7)
- added JP2: JP_GND, Jumper:SolderJumper-2_P1.3mm_Open_Pad1.0x1.5mm, F.Cu at (97.9, 54.2)
- added JP3: JP_RST, Jumper:SolderJumper-2_P1.3mm_Open_Pad1.0x1.5mm, F.Cu at (97.9, 57.8)
- added JP4: Jumper_2_Open, Jumper:SolderJumper-2_P1.3mm_Bridged_Pad1.0x1.5mm, F.Cu at (97.9, 61.4)
- added L1: 10uH, Inductor_SMD:L_1206_3216Metric_Pad1.42x1.75mm_HandSolder, F.Cu at (82.9, 83.9)
- added M1: M1_Conn_Alt, MM_Library:Motor Headers, F.Cu at (71.8, 93.5)
- added M2: M2_Conn_Alt, MM_Library:Motor Headers, F.Cu at (71.8, 105.4)
- added MOS1: SSM3K335R_LF, custom_foot:SOT-23F_TOS, F.Cu at (103.7, 65.4)
- added M_MH1: M2, MM_Library:Motor_mouse, F.Cu at (61.8, 31.2)
- added M_MH2: M2, MM_Library:Motor_mouse, F.Cu at (61.8, 60.4)
- added Q0: TEFT4300, MM_Library:Emitter, F.Cu at (86.4, 72.4)
- added Q1: TEFT4300, MM_Library:Emitter, F.Cu at (92.0, 72.4)
- added Q10: Q_NMOS_GSD, Package_TO_SOT_SMD:SOT-23, F.Cu at (35.7, 98.0)
- added Q11: Q_NMOS_GSD, Package_TO_SOT_SMD:SOT-23, F.Cu at (35.7, 102.4)
- added Q12: Q_NMOS_GSD, Package_TO_SOT_SMD:SOT-23, F.Cu at (35.7, 106.8)
- added Q2: TEFT4300, MM_Library:Emitter, F.Cu at (97.6, 72.4)
- added Q3: TEFT4300, MM_Library:Emitter, F.Cu at (103.2, 72.4)
- added Q8: Q_NMOS_SGD, Package_TO_SOT_SMD:SOT-23, F.Cu at (35.7, 89.0)
- added Q9: Q_NMOS_GSD, Package_TO_SOT_SMD:SOT-23, F.Cu at (35.7, 93.5)
- added R1: 1.8k, Resistor_SMD:R_1206_3216Metric_Pad1.30x1.75mm_HandSolder, F.Cu at (82.9, 87.2)
- added R11: 47K, Resistor_SMD:R_1206_3216Metric_Pad1.30x1.75mm_HandSolder, F.Cu at (88.8, 97.0)
- added R12: 47K, Resistor_SMD:R_1206_3216Metric_Pad1.30x1.75mm_HandSolder, F.Cu at (88.8, 100.3)
- added R13: 47k, Resistor_SMD:R_1206_3216Metric_Pad1.30x1.75mm_HandSolder, F.Cu at (94.8, 83.9)
- added R14: 47k, Resistor_SMD:R_1206_3216Metric_Pad1.30x1.75mm_HandSolder, F.Cu at (94.8, 87.2)
- added R15: 47k, Resistor_SMD:R_1206_3216Metric_Pad1.30x1.75mm_HandSolder, F.Cu at (94.8, 90.4)
- added R16: 47k, Resistor_SMD:R_1206_3216Metric_Pad1.30x1.75mm_HandSolder, F.Cu at (94.8, 93.7)
- added R17: 47k, Resistor_SMD:R_1206_3216Metric_Pad1.30x1.75mm_HandSolder, F.Cu at (94.8, 97.0)
- added R18: 0, Resistor_SMD:R_1206_3216Metric_Pad1.30x1.75mm_HandSolder, F.Cu at (94.8, 100.3)
- added R19: 750, Resistor_SMD:R_1206_3216Metric_Pad1.30x1.75mm_HandSolder, F.Cu at (100.7, 83.9)
- added R2: 1.8k, Resistor_SMD:R_1206_3216Metric_Pad1.30x1.75mm_HandSolder, F.Cu at (82.9, 90.4)
- added R20: 75, Resistor_SMD:R_1206_3216Metric_Pad1.30x1.75mm_HandSolder, F.Cu at (100.7, 87.2)
- added R21: 75, Resistor_SMD:R_1206_3216Metric_Pad1.30x1.75mm_HandSolder, F.Cu at (100.7, 90.4)
- added R22: 20K, Resistor_SMD:R_1206_3216Metric_Pad1.30x1.75mm_HandSolder, F.Cu at (100.7, 93.7)
- added R23: 10K, Resistor_SMD:R_1206_3216Metric_Pad1.30x1.75mm_HandSolder, F.Cu at (100.7, 97.0)
- added R24: 47K, Resistor_SMD:R_1206_3216Metric_Pad1.30x1.75mm_HandSolder, F.Cu at (100.7, 100.3)
- added R3: 1.8k, Resistor_SMD:R_1206_3216Metric_Pad1.30x1.75mm_HandSolder, F.Cu at (82.9, 93.7)
- added R4: 1.8k, Resistor_SMD:R_1206_3216Metric_Pad1.30x1.75mm_HandSolder, F.Cu at (82.9, 97.0)
- added R5: 35, Resistor_SMD:R_1206_3216Metric_Pad1.30x1.75mm_HandSolder, F.Cu at (82.9, 100.3)
- added R6: 35, Resistor_SMD:R_1206_3216Metric_Pad1.30x1.75mm_HandSolder, F.Cu at (88.8, 83.9)
- added R7: 35, Resistor_SMD:R_1206_3216Metric_Pad1.30x1.75mm_HandSolder, F.Cu at (88.8, 87.2)
- added R8: 35, Resistor_SMD:R_1206_3216Metric_Pad1.30x1.75mm_HandSolder, F.Cu at (88.8, 90.4)
- added R9: 47K, Resistor_SMD:R_1206_3216Metric_Pad1.30x1.75mm_HandSolder, F.Cu at (88.8, 93.7)
- added S1: EG1218, MM_Library:MM Switch, F.Cu at (46.2, 83.9)
- added SK1: M2, MountingHole:MountingHole_2.2mm_M2, F.Cu at (30.1, 77.9)
- added SK2: M2, MountingHole:MountingHole_2.2mm_M2, F.Cu at (30.1, 83.8)
- added SK3: M2, MountingHole:MountingHole_2.2mm_M2, F.Cu at (36.0, 77.9)
- added SK4: M2, MountingHole:MountingHole_2.2mm_M2, F.Cu at (36.0, 83.8)
- added SW1: SW, Button_Switch_SMD:SW_SPST_REED_CT05-XXXX-G1, F.Cu at (44.5, 89.3)
- added SW2: SW, Button_Switch_SMD:SW_SPST_REED_CT05-XXXX-G1, F.Cu at (44.5, 94.4)
- added SW3: SW, Button_Switch_SMD:SW_SPST_REED_CT05-XXXX-G1, F.Cu at (44.5, 99.5)
- added SW_RST1: SW, Button_Switch_SMD:SW_SPST_REED_CT05-XXXX-G1, F.Cu at (44.5, 104.5)
- added TP1: V_EXT_TP, Connector_PinHeader_2.54mm:PinHeader_1x01_P2.54mm_Vertical, F.Cu at (82.2, 104.3)
- added TP2: GND_TP, Connector_PinHeader_2.54mm:PinHeader_1x01_P2.54mm_Vertical, F.Cu at (82.2, 108.9)
- added TP3: TP_5V, Connector_PinHeader_2.54mm:PinHeader_1x01_P2.54mm_Vertical, F.Cu at (86.9, 104.3)
- added TP4: TP_3V3, Connector_PinHeader_2.54mm:PinHeader_1x01_P2.54mm_Vertical, F.Cu at (86.9, 108.9)
- added TP5: GND_TP, Connector_PinHeader_2.54mm:PinHeader_1x01_P2.54mm_Vertical, F.Cu at (91.5, 104.3)
- added TP6: GND_TP, Connector_PinHeader_2.54mm:PinHeader_1x01_P2.54mm_Vertical, F.Cu at (91.5, 108.9)
- added U1: YAAJ_BluePill_SWD_Breakout, MM_Library:STM32F103, F.Cu at (74.2, 42.3)
- added U2: TB6612FNG, Package_SO:SSOP-24_5.3x8.2mm_P0.65mm, F.Cu at (56.1, 91.8)
- added U3: LM1085-5.0, MM_Library:5V Voltage Reg, F.Cu at (95.3, 30.8)
- added U4: APE8865Y5-33-HF-3, Package_TO_SOT_SMD:SOT-23-5, F.Cu at (89.0, 66.0)
- added U5: LM66100DCKR, custom_foot:DCK6_TEX, F.Cu at (101.7, 103.9)
- added U6: LM66100DCKR, custom_foot:DCK6_TEX, F.Cu at (101.7, 107.7)

Commit message: Completed routing for version using bluepill, no DRC errors. Began routing for version with no bluepill
Parts:
- removed BT_MH1, BT_MH2, BT_MH3, BT_MH4: M2, MountingHole:MountingHole_2.2mm_M2
- C1, C19, C25, C6, C8, C9, FB3, FB4, JP1, JP2, JP3, Q8, R11, R12, R15, R17, R18, R22, R23, R24, R9, U4: moved to B.Cu
- Q0, Q1, Q2, Q3: value TEFT4300 -> Q_Photo_NPN
- moved C1 223.2 mm to (240.2, 111.8), turned to 90 degrees
- moved C9 219.5 mm to (237.6, 111.8), turned to -90 degrees
- moved Q9 216.6 mm to (241.5, 161.2)
- moved C12 215.6 mm to (221.8, 178.2), turned to -90 degrees
- moved C11 214.4 mm to (219.0, 178.2), turned to -90 degrees
- moved C18 211.9 mm to (224.4, 178.2), turned to -90 degrees
- moved C25 211.2 mm to (227.8, 173.2), turned to 180 degrees
- moved SW1 207.3 mm to (243.2, 148.4)
- moved SW2 207.1 mm to (243.2, 152.7)
- moved SW3 206.9 mm to (243.2, 156.8)
- moved SK4 202.0 mm to (207.0, 191.4)
- moved SK3 201.0 mm to (207.0, 183.6)
- moved D0 200.9 mm to (242.7, 164.4)
- moved C17 200.7 mm to (224.4, 120.0), turned to 180 degrees
- moved S1 195.3 mm to (240.1, 107.2), turned to -90 degrees
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- renumbered SW_RST1 to RESET
Connections:
- R22 pad 1: BATT_NET -> VCC
Routing:
- net RST: track 0.00 -> 150.5 mm, vias 0 -> 3
- net LED_RED: track 0.00 -> 104.4 mm, vias 0 -> 4
- net LED_BLUE: track 0.00 -> 103.6 mm, vias 0 -> 4
- net LED_GREEN: track 0.00 -> 99.8 mm, vias 0 -> 4
- net +3.3VA: track 0.00 -> 92.9 mm
- net VCC: track 0.00 -> 92.6 mm, vias 0 -> 5
- net +3V3: track 0.00 -> 89.4 mm, vias 0 -> 6
- net M1_SPD: track 0.00 -> 80.0 mm, vias 0 -> 1
- net +5V_NET: track 0.00 -> 75.3 mm, vias 0 -> 2
- net BLE_STATE: track 0.00 -> 73.2 mm
- net Net-(J1-Pin_2): track 0.00 -> 62.9 mm, vias 0 -> 2
- net BUTTON_2: track 0.00 -> 60.8 mm, vias 0 -> 3
- net BUZZER: track 0.00 -> 60.6 mm, vias 0 -> 1
- net +3V3_NET: track 0.00 -> 58.5 mm, vias 0 -> 1
- net BUTTON_3: track 0.00 -> 56.5 mm, vias 0 -> 3
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- added copper zone on In1.Cu, net +3V3
- added copper zone on In1.Cu, net +5V
- added copper zone on B.Cu, net GND
- added copper zone on F.Cu, net GND
- added copper zone on In2.Cu, net GND
Other:
- board outline added: 84.9 x 94.9 mm
- copper layers 2 -> 4
- board text added: "+3V3"
- board text added: "+3V3 SWDIO SWDCLK GND"
- board text added: "+5V"
- board text added: "- +"
- board text added: "B"
- board text added: "BLE TX RX GND +5V"
- board text added: "G"
- board text added: "GND"
- board text added: "R"
- board text added: "TX RX GND"
- board text added: "VCC"

Commit message: Completed routing of non-bluepill version of schematic. All DRC errors cleared. Version/Name/Year label updated. To be reviewed.
Routing:
- net GND: vias 8 -> 9
Other:
- board text added: "J. Low, T. Tang N. Ward v0.4 2024"
Changed lines of the file:
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@@
     )
   )
+  (gr_line (start 217.2 128.06506) (end 197.49976 128.06506)
+    (stroke (width 0.2) (type solid)) (layer "B.SilkS"))
+  (gr_line (start 197.515 120.44506) (end 217.23556 120.43236)
+    (stroke (width 0.2) (type solid)) (layer "B.SilkS"))
+  (gr_line (start 217.2 120.6) (end 217.2 128.06506)
+    (stroke (width 0.2) (type solid)) (layer "B.SilkS"))
+  (gr_line (start 197.515 128.06506) (end 197.515 120.44506)
+    (stroke (width 0.2) (type solid)) (layer "B.SilkS"))
   (gr_line (start 167.74538 98.34068) (end 245.92912 98.33306)
     (stroke (width 0.15) (type solid)) (layer "Edge.Cuts"))
@@
   (gr_line (start 164.43576 167.16452) (end 164.4256 145.8463)
     (stroke (width 0.15) (type solid)) (layer "Edge.Cuts"))
+  (gr_text "J. Low, T. Tang\nN. Ward\nv0.4  2024" (at 207.04 124.25506 180) (layer "B.SilkS")
+    (effects (font (size 1.5 1.5) (thickness 0.3)) (justify mirror))
+  )
   (gr_text "+5V\n" (at 196 100) (layer "F.SilkS")
     (effects (font (size 1 1) (thickness 0.15)) (justify left bottom))
@@
   (via (at 211 115.2) (size 0.8) (drill 0.4) (layers "F.Cu" "B.Cu") (free) (net 2))
   (via (at 234.7 131.1) (size 0.8) (drill 0.4) (layers "F.Cu" "B.Cu") (free) (net 2))
+  (via (at 185.9 158.1) (size 0.8) (drill 0.4) (layers "F.Cu" "B.Cu") (free) (net 2))
   (via (at 196 131) (size 0.8) (drill 0.4) (layers "F.Cu" "B.Cu") (free) (net 2))
   (via (at 185.3 182.2) (size 0.8) (drill 0.4) (layers "F.Cu" "B.Cu") (free) (net 2))
