File: PCB/bare_mouse/bloo.kicad_pcb (KiCad board)
At the start: 4 copper layers, 84.9 x 94.9 mm, 101 parts, among them J1 Serial Debug Header, J10 Conn_01x06_Female, J2 SWD Header, J4 Conn_ARM_JTAG_SWD_10, J5 SWD Header, M1 M1_Conn_Alt, M2 M2_Conn_Alt, Q0 Q_Photo_NPN, Q1 Q_Photo_NPN, Q10 Q_NMOS_GSD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

Commit message: Updated bluepill version of mouse to use L293D motor driver rather than TB6612FNG
Parts:
- removed C5: 0.1uF, Capacitor_SMD:C_1206_3216Metric_Pad1.33x1.80mm_HandSolder
- removed C7: 10uF, Capacitor_SMD:C_1206_3216Metric_Pad1.33x1.80mm_HandSolder
- C3: value 10uF -> 1uF
- U2: value TB6612FNG -> L293D; footprint Package_SO:SSOP-24_5.3x8.2mm_P0.65mm -> Package_DIP:DIP-16_W7.62mm
- moved U2 20.9 mm to (201.0, 122.4), turned to 90 degrees
- moved C3 19.8 mm to (209.0, 141.4)
- moved C4 19.5 mm to (204.6, 141.3)
- moved J1 0.10 mm to (189.7, 110.7)
- renumbered RESET to SW_RST1
Connections:
- C4 pad 1: VCC -> +5V
- U2 pad 1: M1_OUT_1 -> M1_SPD
- U2 pad 10: GND -> M2_FWD
- U2 pad 12: M2_OUT_1 -> GND
- U2 pad 13: VCC -> GND
- U2 pad 14: VCC -> M2_OUT_2
- U2 pad 15: M2_SPD -> M2_BACK
- U2 pad 16: M2_BACK -> +5V
- U2 pad 2: M1_OUT_1 -> M1_FWD
- U2 pad 3: GND -> M1_OUT_1
- U2 pad 5: M1_OUT_2 -> GND
- U2 pad 7: M2_OUT_2 -> M1_BACK
- U2 pad 8: M2_OUT_2 -> VCC
- U2 pad 9: GND -> M2_SPD
Routing:
- net M2_SPD: track 29.5 -> 90.2 mm, vias 1 -> 2
- net M2_BACK: track 25.2 -> 60.9 mm
- net M1_SPD: track 80.0 -> 45.9 mm, vias 1 -> 0
- net VCC: track 92.6 -> 61.7 mm, vias 5 -> 3
- net M2_OUT_1: track 29.8 -> 53.8 mm, vias 2 -> 0
- net M2_FWD: track 26.9 -> 44.3 mm, vias 2 -> 0
- net M2_OUT_2: track 23.0 -> 38.9 mm
- net M1_BACK: track 46.0 -> 37.1 mm, vias 1 -> 0
- net +5V: track 29.3 -> 21.2 mm, vias 6 -> 5
- net +5V_NET: track 75.3 -> 70.8 mm
- net M1_OUT_2: track 29.2 -> 27.3 mm
- net M1_FWD: track 41.8 -> 40.0 mm, vias 1 -> 0
- net Net-(J1-Pin_3): track 53.1 -> 52.1 mm
- net M1_OUT_1: track 30.7 -> 31.3 mm
- net GND: track 0.40 -> 0.00 mm, vias 9 -> 15
