File: PCB/bare_mouse_nobluepill/bloo.kicad_pcb (KiCad board)
At the start: 2 copper layers, 114 parts, among them J1 Serial Debug Header, J10 Conn_01x06_Female, J2 SWD Header, J4 Conn_ARM_JTAG_SWD_10, J5 SWD Header, M1 M1_Conn_Alt, M2 M2_Conn_Alt, Q0 TEFT4300, Q1 TEFT4300, Q10 Q_NMOS_GSD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

Commit message: Completed routing for version using bluepill, no DRC errors. Began routing for version with no bluepill
Parts:
- removed BT_MH1, BT_MH2, BT_MH3, BT_MH4: M2, MountingHole:MountingHole_2.2mm_M2
- removed J5: SWD Header, Connector_PinHeader_2.54mm:PinHeader_1x05_P2.54mm_Vertical
- removed SW_RST1: SW, Button_Switch_SMD:SW_SPST_REED_CT05-XXXX-G1
- added POWER: LED, LED_SMD:LED_0805_2012Metric_Pad1.15x1.40mm_HandSolder, F.Cu at (184.1, 151.7)
- added R26: 750, Resistor_SMD:R_1206_3216Metric_Pad1.30x1.75mm_HandSolder, F.Cu at (179.5, 151.6)
- added RESET: SW, Button_Switch_SMD:SW_SPST_REED_CT05-XXXX-G1, F.Cu at (184.9, 96.5)
- C1, C19, C25, C6, C8, C9, FB3, FB4, JP1, JP2, JP3, Q8, R10, R17, R18, R22, R23, R25, U4: moved to B.Cu
- Q0, Q1, Q2, Q3: value TEFT4300 -> Q_Photo_NPN
- moved D0 227.9 mm to (237.3, 160.5)
- moved Q0 204.8 mm to (231.9, 166.7)
- moved C11 203.8 mm to (213.7, 174.3), turned to -90 degrees
- moved C12 203.2 mm to (216.5, 174.3), turned to -90 degrees
- moved D1 203.0 mm to (203.8, 184.2), turned to 63.5 degrees
- moved C18 193.1 mm to (219.1, 174.3), turned to -90 degrees
- moved Q1 189.2 mm to (211.4, 181.7), turned to 63.5 degrees
- moved U3 189.2 mm to (220.7, 92.7), turned to 180 degrees
- moved C25 187.7 mm to (222.5, 169.3), turned to 180 degrees
- moved D3 187.7 mm to (198.3, 181.9), turned to -63.5 degrees
- moved L1 185.6 mm to (225.1, 175.0)
- moved C1 183.5 mm to (234.9, 107.9), turned to 90 degrees
- moved R5 182.7 mm to (240.9, 157.3), turned to 180 degrees
- moved C2 181.7 mm to (234.1, 101.9), turned to 180 degrees
- moved TP2 176.7 mm to (230.3, 141.9)
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Connections:
- R22 pad 1: BATT_NET -> VCC
- U7 pad 2: unconnected-(U7-PC13-Pad2) -> POWER_LED
Routing:
- added copper zone on In1.Cu, net +3V3
- added copper zone on In1.Cu, net +5V
- added copper zone on B.Cu, net GND
- added copper zone on F.Cu, net GND
- added copper zone on In2.Cu, net GND
Other:
- board outline added: 84.9 x 94.9 mm
- copper layers 2 -> 4
- board text added: "+3V3"
- board text added: "+3V3 SWDIO SWDCLK GND"
- board text added: "+5V"
- board text added: "- +"
- board text added: "B"
- board text added: "BLE TX RX GND +5V"
- board text added: "G"
- board text added: "GND"
- board text added: "R"
- board text added: "TX RX GND"
- board text added: "VCC"

Commit message: Completed routing of non-bluepill version of schematic. All DRC errors cleared. Version/Name/Year label updated. To be reviewed.
Parts:
- moved JP1 1.31 mm to (170.5, 153.8)
- moved C28 1.20 mm to (194.7, 169.4)
- moved C29 1.20 mm to (192.1, 169.4)
- moved FB3 0.90 mm to (213.0, 154.1)
- moved R9 0.60 mm to (227.4, 152.4)
- moved R11 0.40 mm to (227.4, 145.2)
- moved R24 0.10 mm to (227.4, 148.8)
- moved R25 0.10 mm to (203.7, 164.6)
- moved C24 0.10 mm to (212.7, 145.7)
- moved R10 0.10 mm to (199.0, 145.3)
Routing:
- net +3.3VA: track 0.00 -> 126.1 mm, vias 0 -> 2
- net LED_BLUE: track 0.00 -> 122.3 mm, vias 0 -> 3
- net LED_RED: track 0.00 -> 115.6 mm, vias 0 -> 3
- net +3V3: track 0.00 -> 114.1 mm, vias 0 -> 10
- net RST: track 0.00 -> 112.7 mm, vias 0 -> 4
- net BUTTON_2: track 0.00 -> 100.2 mm, vias 0 -> 2
- net VCC: track 0.00 -> 97.9 mm, vias 0 -> 5
- net LED_GREEN: track 0.00 -> 79.2 mm, vias 0 -> 2
- net +5V_NET: track 0.00 -> 74.9 mm, vias 0 -> 2
- net BLE_STATE: track 0.00 -> 71.7 mm, vias 0 -> 2
- net BUZZER: track 0.00 -> 71.4 mm, vias 0 -> 1
- net Net-(J1-Pin_2): track 0.00 -> 70.0 mm, vias 0 -> 2
- net Net-(J1-Pin_3): track 0.00 -> 64.7 mm, vias 0 -> 2
- net M2_FWD: track 0.00 -> 61.1 mm, vias 0 -> 2
- net SWDCLK: track 0.00 -> 60.8 mm, vias 0 -> 1
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Other:
- board text added: "J. Low, T. Tang N. Ward v0.4 2024"
